File: fen.brd (EAGLE design)
At the start: 64.4 x 35.5 mm, 75 parts, among them Q1 MOSFET-NCHANNELFDD8780, Q3 TRANSISTOR_PNPSMD, T1 BT138-H, U1 STM32F042FX, Y1 8MHZ

Commit message: change board
Parts:
- moved JP7 1.31 mm to (3.05, 18.0)
- moved JP6 1.19 mm to (3.05, 20.7)
- moved R28 0.30 mm to (8.89, 16.8)
- moved R29 0.30 mm to (12.7, 16.8)
- moved U$2 0.30 mm to (23.2, 24.1)
- moved R19 0.30 mm to (6.05, 21.1)
- moved R21 0.30 mm to (6.05, 19.1)
- moved R16 0.22 mm to (4.93, 30.6)
Routing:
- net VCC: track 102.6 -> 115.4 mm
- net GND: track 68.4 -> 61.3 mm, vias 10 -> 9
- net SCL: track 35.2 -> 37.5 mm, vias 2 -> 1
- net VCC-IN: track 67.2 -> 68.9 mm
- net SDA: track 35.6 -> 37.2 mm
- net N$21: track 10.5 -> 11.7 mm
- net N$23: track 4.19 -> 5.14 mm
- net N$22: track 3.77 -> 4.48 mm
- net N: track 51.7 -> 52.4 mm
